File: poe32net-original-v0.1.kicad_pcb (KiCad board)
At the start: 2 copper layers, 70 x 90 mm, 76 parts, among them J1 RJ45_LED_Shielded, J10 01x03, J11 01x03, J12 01x03, J13 01x03, J14 01x03, J15 01x03, J16 01x03, J17 01x03, J18 01x03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

Commit message: v0.2
Parts:
- added D5: D_Schottky, Diode_SMD:D_SOD-128, F.Cu at (139.6, 103.4)
- added D6: D_Schottky, Diode_SMD:D_SOD-128, F.Cu at (165.6, 109.2)
- moved J4 89.2 mm to (192.7, 92.4), turned to 0 degrees
- moved J3 88.4 mm to (188.1, 92.4), turned to 0 degrees
- moved J7 88.0 mm to (197.4, 107.2), turned to 0 degrees
- moved J6 87.2 mm to (192.7, 107.2), turned to 0 degrees
- moved J5 86.5 mm to (188.1, 107.2), turned to 0 degrees
- moved C2 43.2 mm to (92.0, 64.7)
- moved C1 43.0 mm to (92.0, 61.3)
- moved R5 37.0 mm to (87.0, 61.1)
- moved R9 30.5 mm to (87.0, 72.9), turned to 0 degrees
- moved Y1 28.1 mm to (105.9, 66.1)
- moved R10 28.0 mm to (87.0, 75.9), turned to 0 degrees
- moved C4 27.9 mm to (92.0, 71.4)
- moved C5 27.4 mm to (92.0, 74.7), turned to 0 degrees
- moved C3 24.8 mm to (92.0, 68.0)
- moved R8 24.0 mm to (87.0, 70.0), turned to 0 degrees
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Routing:
- net +3V3: track 362.7 -> 264.6 mm, vias 7 -> 5
- net /ETH-TXD1: track 64.1 -> 0.00 mm, vias 2 -> 0
- net /ETH-TXEN: track 57.8 -> 0.00 mm, vias 2 -> 0
- net /ETH-TXD0: track 53.4 -> 0.00 mm, vias 2 -> 0
- net /ETH-MDIO: track 53.0 -> 0.00 mm, vias 2 -> 0
- net /ETH-MDC: track 77.3 -> 26.6 mm
- net Net-(U3-~{RST}): track 51.0 -> 1.61 mm
- net /ETH-RCLK: track 46.8 -> 0.00 mm, vias 2 -> 0
- net /ETH-CRS: track 36.0 -> 0.18 mm, vias 2 -> 0
- net GND: track 303.4 -> 269.4 mm, vias 19 -> 14
- net /ETH-RXD0: track 28.7 -> 0.00 mm
- net /GPIO32: track 27.9 -> 0.00 mm, vias 1 -> 0
- net /GPIO35: track 26.8 -> 0.00 mm, vias 1 -> 0
- net /GPIO33: track 26.8 -> 0.00 mm, vias 1 -> 0
- net /ETH-RXD1: track 26.6 -> 0.00 mm
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- removed copper zone on B.Cu, net GND
- removed copper zone on F.Cu, net GND
Other:
- board text removed: "34"
- board text removed: "35"
