File: poe32net-original-v0.1.kicad_sch (KiCad schematic)
At the start: 76 parts, among them J1 RJ45_LED_Shielded, J10 01x03, J11 01x03, J12 01x03, J13 01x03, J14 01x03, J15 01x03, J16 01x03, J17 01x03, J18 01x03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

Commit message: v0.2
Parts:
- added D5, D6: D_Schottky, Diode_SMD:D_SOD-128, symbol Device:D_Schottky
Connections:
- net GND: now also D5.2 (A), D6.2 (A)
- net at L1.1, U2.2 (OUT): now also D6.1 (K)
- net at L2.1, U5.2 (OUT): now also D5.1 (K)
Changed lines of the file:
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@@
   (junction (at 107.95 30.48) (diameter 0) (color 0 0 0 0)
   )
+  (junction (at 257.81 116.84) (diameter 0) (color 0 0 0 0)
+  )
   (junction (at 60.96 182.88) (diameter 0) (color 0 0 0 0)
   )
@@
   (junction (at 147.32 33.02) (diameter 0) (color 0 0 0 0)
   )
+  (junction (at 257.81 147.32) (diameter 0) (color 0 0 0 0)
+  )
   (junction (at 243.84 156.21) (diameter 0) (color 0 0 0 0)
   )
@@
   (junction (at 138.43 106.68) (diameter 0) (color 0 0 0 0)
   )
+  (junction (at 257.81 157.48) (diameter 0) (color 0 0 0 0)
+  )
   (junction (at 257.81 48.26) (diameter 0) (color 0 0 0 0)
   )
@@
   (junction (at 260.35 50.8) (diameter 0) (color 0 0 0 0)
   )
+  (junction (at 257.81 127) (diameter 0) (color 0 0 0 0)
+  )
   (junction (at 20.32 171.45) (diameter 0) (color 0 0 0 0)
   )
@@
     (stroke (width 0) (type default))
   )
-  (wire (pts (xy 256.54 116.84) (xy 260.35 116.84))
+  (wire (pts (xy 256.54 116.84) (xy 257.81 116.84))
     (stroke (width 0) (type default))
   )
@@
     (stroke (width 0) (type default))
   )
-  (wire (pts (xy 243.84 157.48) (xy 267.97 157.48))
+  (wire (pts (xy 243.84 157.48) (xy 257.81 157.48))
     (stroke (width 0) (type default))
   )
@@
     (stroke (width 0) (type default))
   )
+  (wire (pts (xy 257.81 156.21) (xy 257.81 157.48))
+    (stroke (width 0) (type default))
+  )
   (wire (pts (xy 46.99 53.34) (xy 46.99 58.42))
     (stroke (width 0) (type default))
@@
     (stroke (width 0) (type default))
   )
+  (wire (pts (xy 257.81 116.84) (xy 257.81 118.11))
+    (stroke (width 0) (type default))
+  )
   (wire (pts (xy 257.81 35.56) (xy 257.81 48.26))
     (stroke (width 0) (type default))
@@
     (stroke (width 0) (type default))
   )
+  (wire (pts (xy 257.81 116.84) (xy 260.35 116.84))
+    (stroke (width 0) (type default))
+  )
   (wire (pts (xy 58.42 179.07) (xy 50.8 179.07))
     (stroke (width 0) (type default))
@@
     (stroke (width 0) (type default))
   )
+  (wire (pts (xy 257.81 147.32) (xy 257.81 148.59))
+    (stroke (width 0) (type default))
+  )
   (wire (pts (xy 38.1 25.4) (xy 38.1 27.94))
     (stroke (width 0) (type default))
@@
     (stroke (width 0) (type default))
   )
+  (wire (pts (xy 257.81 147.32) (xy 260.35 147.32))
+    (stroke (width 0) (type default))
+  )
   (wire (pts (xy 95.25 175.26) (xy 100.33 175.26))
     (stroke (width 0) (type default))
@@
     (stroke (width 0) (type default))
   )
+  (wire (pts (xy 257.81 157.48) (xy 267.97 157.48))
+    (stroke (width 0) (type default))
+  )
   (wire (pts (xy 13.97 144.78) (xy 13.97 156.21))
     (stroke (width 0) (type default))
@@
     (stroke (width 0) (type default))
   )
-  (wire (pts (xy 243.84 127) (xy 267.97 127))
+  (wire (pts (xy 243.84 127) (xy 257.81 127))
     (stroke (width 0) (type default))
   )
@@
     (stroke (width 0) (type default))
   )
-  (wire (pts (xy 256.54 147.32) (xy 260.35 147.32))
+  (wire (pts (xy 256.54 147.32) (xy 257.81 147.32))
     (stroke (width 0) (type default))
   )
@@
     (stroke (width 0) (type default))
   )
+  (wire (pts (xy 257.81 125.73) (xy 257.81 127))
+    (stroke (width 0) (type default))
+  )
   (wire (pts (xy 173.99 55.88) (xy 177.8 55.88))
     (stroke (width 0) (type default))
@@
   )
   (wire (pts (xy 260.35 62.23) (xy 260.35 73.66))
+    (stroke (width 0) (type default))
+  )
+  (wire (pts (xy 257.81 127) (xy 267.97 127))
     (stroke (width 0) (type default))
   )
@@
         (path "/289d480a-a91f-4898-8314-63b2a14b2e7c"
           (reference "J16") (unit 1)
+        )
+      )
+    )
+  )
+  (symbol (lib_id "Device:D_Schottky") (at 257.81 152.4 270) (unit 1)
+    (in_bom yes) (on_board yes) (dnp no) (fields_autoplaced)
+    (property "Reference" "D6" (at 260.35 151.4475 90)
+      (effects (font (size 1.27 1.27)) (justify left))
+    )
+    (property "Value" "D_Schottky" (at 260.35 153.9875 90)
+      (effects (font (size 1.27 1.27)) (justify left))
+    )
+    (property "Footprint" "Diode_SMD:D_SOD-128" (at 257.81 152.4 0)
+      (effects (font (size 1.27 1.27)) hide)
+    )
+    (property "Datasheet" "~" (at 257.81 152.4 0)
+      (effects (font (size 1.27 1.27)) hide)
+    )
+    (property "LCSC" "C65010" (at 257.81 152.4 90)
+      (effects (font (size 1.27 1.27)) hide)
+    )
+    (pin "1")
+    (pin "2")
+    (instances
+      (project "poe32net-original-v0.1"
+        (path "/289d480a-a91f-4898-8314-63b2a14b2e7c"
+          (reference "D6") (unit 1)
         )
       )
@@
         )
       )
+    )
+  )
+  (symbol (lib_id "Device:D_Schottky") (at 257.81 121.92 270) (unit 1)
+    (in_bom yes) (on_board yes) (dnp no) (fields_autoplaced)
+    (property "Reference" "D5" (at 260.35 120.9675 90)
+      (effects (font (size 1.27 1.27)) (justify left))
+    )
+    (property "Value" "D_Schottky" (at 260.35 123.5075 90)
+      (effects (font (size 1.27 1.27)) (justify left))
+    )
+    (property "Footprint" "Diode_SMD:D_SOD-128" (at 257.81 121.92 0)
+      (effects (font (size 1.27 1.27)) hide)
+    )
+    (property "Datasheet" "~" (at 257.81 121.92 0)
+      (effects (font (size 1.27 1.27)) hide)
+    )
+    (property "LCSC" "C65010" (at 257.81 121.92 90)
+      (effects (font (size 1.27 1.27)) hide)
+    )
+    (pin "1")
+    (pin "2")
+    (instances
+      (project "poe32net-original-v0.1"
+        (path "/289d480a-a91f-4898-8314-63b2a14b2e7c"
+          (reference "D5") (unit 1)
+        )
+      )
